File: BirdBuildingBlock.brd (EAGLE design)
At the start: 31.2 x 30.7 mm, 45 parts, among them CN2 JSTPH, CN3 AMP FCI 10103594-0001LF, U1 UG-2828GDEDF11, U2 MIC5225-3.3v, U3 FAN5331SX, U4 CH340G, U6 MCP73831T-2ACI/OT, Y2 12MHz

Commit message: Finalizing some circuit design and cleaning up the pcb layout
Parts:
- removed C11: 0.1uF, adafruit:C0805
- removed C15: 10uF, adafruit:C0805
- removed D4: SCHOTTKY, adafruit:SOD-123FL
- removed J1: (no value), SparkFun-Connectors:1X02
- removed U5: (no value), esp8266modules:ESP12-SMD
- added Q1, Q2: mmbt2222, SparkFun:SOT23-3
- added R2, R3: 10K, adafruit:R0603
- added R8: 10K, microbuilder:0805
- added X1: (no value), adafruit:ESP-12
- moved C17 96.2 mm to (5.84, 19.7), turned to 180 degrees
- moved C14 94.4 mm to (20.3, 20.8)
- moved Y2 93.9 mm to (20.6, 18.3)
- moved C16 93.4 mm to (13.2, 15.7)
- moved C9 89.9 mm to (20.3, 15.7), turned to 180 degrees
- moved D5 89.1 mm to (4.19, 26.2), flipped to the bottom, turned to 180 degrees
- moved U4 88.8 mm to (13.0, 20.6)
- moved CHG 88.5 mm to (1.52, 23.1), flipped to the bottom, turned to 180 degrees
- moved S1 88.0 mm to (6.10, 28.8)
- moved R13 84.1 mm to (9.40, 26.2), flipped to the bottom
- moved U6 82.1 mm to (4.57, 19.8), flipped to the bottom
- moved C12 81.1 mm to (22.6, 26.0)
- moved R9 80.1 mm to (4.19, 23.1), flipped to the bottom
- moved R1 77.7 mm to (1.52, 19.4), flipped to the bottom, turned to 270 degrees
- moved CN2 75.5 mm to (2.16, 13.2), turned to 90 degrees
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Connections:
- removed net !CTS: U4.9
- removed net !DTR: U4.13
- removed net N$15: R12.1, U5.GPIO0
- removed net N$16: R10.2, U5.CH_PD
- removed net N$18: J1.2, U5.GPIO12
- removed net N$2: R11.2, U5.RESET
- removed net RXI: U4.3
- removed net TXO: U4.2
- removed net VIN: C15.1, C6.1, D4.C, D5.C, U2.1, U2.3
- new net CH_PD: R10.2, X1.3
- new net D+: CN3.D+, U4.5
- new net D-: CN3.D-, U4.6
- new net DTR: Q2.2, R2.1, U4.13
- new net GPIO0: Q2.3, R12.1, X1.12
- new net RESET: Q1.3, R11.2, X1.1
- new net RTS: Q1.2, R3.1, U4.14
- net +3V3: now also X1.8; no longer C11.1, U5.VCC
- net GND: now also R8.1, X1.9; no longer C11.2, C15.2, J1.1, U5.GND
- net MOSI/DATA1: now also X1.7; no longer U5.GPIO13
- net N$13: now also Q1.1, R2.2; no longer U4.6
- net N$14: now also Q2.1, R3.2; no longer U4.5
- net N$17: now also X1.10; no longer U5.GPIO15
- net OLED_BS0: now also R8.2
- net OLED_CS: now also X1.4; no longer U5.GPIO16
- net OLED_DC: now also X1.14; no longer U5.GPIO4
- net OLED_RES: now also X1.13; no longer U5.GPIO5
- net RX: now also U4.2, X1.15; no longer U5.RXD0
- net SCK/DATA0: now also X1.5; no longer U5.GPIO14
- net TX: now also U4.3, X1.16; no longer U5.TXD0
- net VBUS: now also C6.1, D5.C, U2.1, U2.3; no longer D4.A
Other:
- board size 31.2 x 30.7 mm -> 31.1 x 30.9 mm
